Commit message: Keyboard reader installitud

File: src/my_r2d2/urdf/r2d2_xacro.urdf.xacro (robot description, xacro)
@@ -224,3 +224,10 @@
     <origin xyz="0 0 ${bodylen/2+wheeldiam+.1}"/>
   </joint>
+  <link name="eye">
+  </link>
+  <joint name="eye_to_box" type="fixed">
+    <parent link= "box" />
+    <child link= "eye" />
+    <origin xyz="0 0 0" rpy="1.57 3.14 1.57" />
+  </joint>
 </robot>
